File: nRF51822.sch (EAGLE design)
At the start: 13 parts

Commit message: Battery
Parts:
- added BAT1: (no value), SparkFun-Electromechanical:BATTERY20SMD
Changed lines of the file:
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@@
 <part name="GND13" library="SparkFun-Aesthetics" deviceset="GND" device=""/>
 <part name="U$2" library="NordicSemi" deviceset="CRYSTAL2.5X2" device=""/>
+<part name="BAT1" library="SparkFun-Electromechanical" deviceset="BATTERY" device="20SMD"/>
 </parts>
 <sheets>
@@
 <instance part="GND13" gate="1" x="68.58" y="101.6"/>
 <instance part="U$2" gate="G$1" x="93.98" y="111.76"/>
+<instance part="BAT1" gate="G$1" x="157.48" y="71.12" rot="R270"/>
 </instances>
 <busses>
