File: nRF51822.sch (EAGLE design)
At the start: 29 parts

Commit message: Board 90%
Parts:
- removed BAT1: (no value), SparkFun-Electromechanical:BATTERY20SMD
- removed S1, S2: (no value), SparkFun-Electromechanical:TAC_SWITCHSMD
- added BATT: 20mm coincell, SparkFun-Electromechanical:BATTERY20MM_4LEGS_OVERPASTE
- added JP: JUMP_SMD, NordicSemi:JUMP_SMD
- added SW1: SWITCH_SMD_BB, NordicSemi:SWITCH_SMD_BB
- added SW2: SW1, NordicSemi:SWITCH_SMD_BB
- renumbered JP1 to PROG, JP2 to EXP, U$1 to NRF51822, U$2 to XT, U$3 to BLN, U$4 to ANT
Connections:
- new net N$7: D1.A, JP.2
- net GND: now also BATT.-, SW1.1, SW2.1; no longer BAT1.-, NRF51822.P0.21, NRF51822.P0.22, NRF51822.P0.23, NRF51822.P0.24, NRF51822.P0.25, S1.1, S1.2, S2.1, S2.2
- net N$16: now also BATT.+, JP.1; no longer BAT1.+, D1.A
- net SW1: now also SW1.2; no longer S1.3, S1.4
- net SW2: now also SW2.2; no longer S2.3, S2.4
Other:
- moved on the sheet: C9, D1

Commit message: BLE NRF51822v1
Board 100%, Lbr update Top places
Connections:
- new net N$17: NRF51822.P0.30
- new net N$21: NRF51822.P0.00
- new net N$24: NRF51822.P0.25
- new net N$25: NRF51822.P0.24
- new net N$26: NRF51822.P0.23
- new net N$32: NRF51822.P0.22
- new net N$33: NRF51822.P0.21
- net GND: no longer NRF51822.P0.00, NRF51822.P0.30
Changed lines of the file:
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@@
 <part name="GND5" library="SparkFun-Aesthetics" deviceset="GND" device=""/>
 <part name="GND6" library="SparkFun-Aesthetics" deviceset="GND" device=""/>
-<part name="GND8" library="SparkFun-Aesthetics" deviceset="GND" device=""/>
 <part name="C4" library="SparkFun-Capacitors" deviceset="CAP" device="0603-CAP" value="47nF"/>
 <part name="C5" library="SparkFun-Capacitors" deviceset="CAP" device="0603-CAP" value="1nF"/>
@@
 <instance part="GND5" gate="1" x="81.28" y="7.62"/>
 <instance part="GND6" gate="1" x="83.82" y="45.72"/>
-<instance part="GND8" gate="1" x="53.34" y="66.04" rot="R270"/>
 <instance part="C4" gate="G$1" x="132.08" y="45.72"/>
 <instance part="C5" gate="G$1" x="132.08" y="71.12"/>
@@
 </segment>
 <segment>
-<pinref part="NRF51822" gate="G$1" pin="P0.30"/>
-<pinref part="GND8" gate="1" pin="GND"/>
-<wire x1="66.04" y1="66.04" x2="63.5" y2="66.04" width="0.1524" layer="91"/>
-<pinref part="NRF51822" gate="G$1" pin="P0.00"/>
-<wire x1="63.5" y1="66.04" x2="55.88" y2="66.04" width="0.1524" layer="91"/>
-<wire x1="66.04" y1="63.5" x2="63.5" y2="63.5" width="0.1524" layer="91"/>
-<wire x1="63.5" y1="63.5" x2="63.5" y2="66.04" width="0.1524" layer="91"/>
-<junction x="63.5" y="66.04"/>
-</segment>
-<segment>
 <pinref part="GND9" gate="1" pin="GND"/>
 <pinref part="C4" gate="G$1" pin="2"/>
@@
 </segment>
 </net>
+<net name="N$24" class="0">
+<segment>
+<pinref part="NRF51822" gate="G$1" pin="P0.25"/>
+<wire x1="91.44" y1="86.36" x2="91.44" y2="88.9" width="0.1524" layer="91"/>
+</segment>
+</net>
+<net name="N$25" class="0">
+<segment>
+<pinref part="NRF51822" gate="G$1" pin="P0.24"/>
+<wire x1="93.98" y1="86.36" x2="93.98" y2="88.9" width="0.1524" layer="91"/>
+</segment>
+</net>
+<net name="N$26" class="0">
+<segment>
+<pinref part="NRF51822" gate="G$1" pin="P0.23"/>
+<wire x1="96.52" y1="86.36" x2="96.52" y2="88.9" width="0.1524" layer="91"/>
+</segment>
+</net>
+<net name="N$32" class="0">
+<segment>
+<pinref part="NRF51822" gate="G$1" pin="P0.22"/>
+<wire x1="99.06" y1="86.36" x2="99.06" y2="88.9" width="0.1524" layer="91"/>
+</segment>
+</net>
+<net name="N$33" class="0">
+<segment>
+<pinref part="NRF51822" gate="G$1" pin="P0.21"/>
+<wire x1="101.6" y1="86.36" x2="101.6" y2="88.9" width="0.1524" layer="91"/>
+</segment>
+</net>
+<net name="N$17" class="0">
+<segment>
+<pinref part="NRF51822" gate="G$1" pin="P0.30"/>
+<wire x1="66.04" y1="66.04" x2="63.5" y2="66.04" width="0.1524" layer="91"/>
+</segment>
+</net>
+<net name="N$21" class="0">
+<segment>
+<pinref part="NRF51822" gate="G$1" pin="P0.00"/>
+<wire x1="66.04" y1="63.5" x2="63.5" y2="63.5" width="0.1524" layer="91"/>
+</segment>
+</net>

Commit message: Esquemático Rev 2
Parts:
- removed D1: BAT165, SparkFun-DiscreteSemi:DIODESOD
- removed EXP: PIN_HEADER_IO, NordicSemi:PIN_HEADER_IO
- removed JP: JUMP_SMD, NordicSemi:JUMP_SMD
- added C13, C14: 12pF, SparkFun-Capacitors:CAP0603-CAP
- added JP1: CM, NordicSemi:JUMP_SMDPITCH_0.05
- added JP2: VCC_PROG, NordicSemi:JUMP_SMDPITCH_0.05
- added P0, P1, P2, P3, P4, P5, P6, P7: TPB1,27, testpad:TPB1,27
- added R4, R5: 4.7K, SparkFun-Resistors:RESISTOR0603-RES
- added R6, R8: 150, SparkFun-Resistors:RESISTOR0603-RES
- added R7, R9: 10K, SparkFun-Resistors:RESISTOR0603-RES
- added T1, T2: BC847, transistor:BC847
- added Y1: CRYSTAL.ABS07, abracon:CRYSTAL.ABS07
- R2, R3: value 100 -> 150
- SW2: value SW1 -> SWITCH_SMD_BB
Connections:
- removed net AIN0: EXP.3, NRF51822.P0.26
- removed net AIN1: EXP.5, NRF51822.P0.27
- removed net AIN2: EXP.7, NRF51822.P0.01
- removed net AIN3: EXP.9, NRF51822.P0.02
- removed net AIN4: EXP.10, NRF51822.P0.03
- removed net AIN5: EXP.8, NRF51822.P0.04
- removed net AIN6: EXP.6, NRF51822.P0.05
- removed net AIN7: EXP.4, NRF51822.P0.06
- removed net N$27 (its old number): NRF51822.P0.07
- removed net SDWCLK: PROG.SWDCLK
- removed net VCC_NRF: C2.1, C3.1, C9.1, D1.C, NRF51822.VDD, NRF51822.VDD_2
- new net N$17: R3.2, T2.C
- new net N$19: R8.2, R9.2, SW2.2
- new net N$34: R4.2, T1.B
- new net N$35: R6.2, R7.2, SW1.2
- new net P00: NRF51822.P0.00, P0.TP
- new net P01: NRF51822.P0.01, P1.TP
- new net P02: NRF51822.P0.02, P2.TP
- new net P03: NRF51822.P0.03, P3.TP
- new net P04: NRF51822.P0.04, P4.TP
- new net P05: NRF51822.P0.05, P5.TP
- new net P06: NRF51822.P0.06, P6.TP
- new net P07: NRF51822.P0.07, P7.TP
- new net XL1: C13.1, NRF51822.P0.26, Y1.2
- new net XL2: C14.1, NRF51822.P0.27, Y1.1
- net GND: now also C13.2, C14.2, JP2.2, T1.E, T2.E; no longer EXP.2
- net LED1: now also R4.1; no longer R2.2
- net LED2: now also R5.1; no longer R3.2
- net N$16: now also JP1.1; no longer JP.1
- net N$21: now also R2.2, T1.C; no longer NRF51822.P0.00
- net N$7: now also R5.2, T2.B; no longer D1.A, JP.2
- net SW1: now also R6.1; no longer SW1.2
- net SW2: now also R8.1; no longer SW2.2
- net SWDCLK: now also PROG.SWDCLK
- net VCC: now also C2.1, C3.1, C9.1, JP1.2, JP2.1, NRF51822.VDD, NRF51822.VDD_2, R7.1, R9.1; no longer EXP.1
Other:
- moved on the sheet: BATT, C10, C11, C9, LED1, LED2, PROG, R2, R3, SW1, SW2
