File: nRF51822.brd (EAGLE design)
At the start: 160 x 100 mm, 24 parts

Commit message: Terminado el Esquemático
Parts:
- added C10, C11: 0.1uF, SparkFun-Capacitors:0603-CAP
- added C12: 2.2nF, SparkFun-Capacitors:0603-CAP
- added U$3: BALUN-2450BM, NordicSemi:2450BM14A0002
- added U$4: ANTENA-2450AT, NordicSemi:2450AT18B100
- JP1: value M05X2SHD_SMD -> PROG-JLINK-SEAGGER; device SparkFun-Connectors:2X5-SHROUDED_SMD -> NordicSemi:M50-3600742
- JP2: value M05X2SHD_SMD -> PIN_HEADER_IO; device SparkFun-Connectors:2X5-SHROUDED_SMD -> NordicSemi:M50-3600742
Connections:
- removed net N$17: JP2.4
- removed net N$20: JP2.3
- removed net N$21: JP2.5
- removed net N$23: JP2.9
- removed net N$24: JP2.6
- removed net N$25: JP2.8
- removed net N$26: JP2.10
- new net ANT1: U$1.31, U$3.4
- new net ANT2: U$1.32, U$3.3
- new net SDWCLK: JP1.4
- new net VDD_PA: C12.1, U$1.30, U$3.5
- net AIN0: now also JP2.3
- net AIN1: now also JP2.5
- net AIN2: now also JP2.7
- net AIN3: now also JP2.9
- net AIN4: now also JP2.10
- net AIN5: now also JP2.8
- net AIN6: now also JP2.6
- net AIN7: now also JP2.4
- net GND: now also C10.2, C11.2, C12.2, U$3.2
- net N$22: now also U$3.1, U$4.FP; no longer JP2.7
- net SWDCLK: no longer JP1.4
- net VCC: now also C10.1, C11.1
Changed lines of the file:
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@@
 <attribute name="PROD_ID" value="SWCH-08247" x="-55.88" y="-20.32" size="1.778" layer="27" display="off"/>
 </element>
-<element name="JP1" library="SparkFun-Connectors" package="2X5-SHROUDED_SMD" value="M05X2SHD_SMD" x="-64.77" y="-11.43"/>
-<element name="JP2" library="SparkFun-Connectors" package="2X5-SHROUDED_SMD" value="M05X2SHD_SMD" x="-74.93" y="-11.43"/>
+<element name="JP1" library="NordicSemi" package="M50-3600742" value="PROG-JLINK-SEAGGER" x="-64.77" y="-11.43"/>
+<element name="JP2" library="NordicSemi" package="M50-3600742" value="PIN_HEADER_IO" x="-74.93" y="-11.43"/>
+<element name="C10" library="SparkFun-Capacitors" package="0603-CAP" value="0.1uF" x="-76.2" y="-25.4"/>
+<element name="C11" library="SparkFun-Capacitors" package="0603-CAP" value="0.1uF" x="-76.2" y="-29.21"/>
+<element name="U$3" library="NordicSemi" package="2450BM14A0002" value="BALUN-2450BM" x="-85.09" y="-25.4"/>
+<element name="U$4" library="NordicSemi" package="2450AT18B100" value="ANTENA-2450AT" x="-92.71" y="-25.4"/>
+<element name="C12" library="SparkFun-Capacitors" package="0603-CAP" value="2.2nF" x="-93.98" y="-33.02"/>
 </elements>
 <signals>
@@
 <contactref element="S2" pad="2"/>
 <contactref element="S2" pad="1"/>
+<contactref element="JP1" pad="3"/>
+<contactref element="JP1" pad="5"/>
 <contactref element="JP1" pad="9"/>
-<contactref element="JP1" pad="5"/>
-<contactref element="JP1" pad="3"/>
 <contactref element="JP2" pad="2"/>
-<wire x1="-67.564" y1="-11.43" x2="-67.564" y2="-16.51" width="0" layer="19" extent="1-1"/>
-<wire x1="-67.564" y1="-8.89" x2="-67.564" y2="-11.43" width="0" layer="19" extent="1-1"/>
-<wire x1="-72.136" y1="-6.35" x2="-67.564" y2="-8.89" width="0" layer="19" extent="1-1"/>
-<wire x1="-58.42" y1="-12.065" x2="-67.564" y2="-11.43" width="0" layer="19" extent="1-1"/>
+<contactref element="C10" pad="2"/>
+<contactref element="C11" pad="2"/>
+<contactref element="C12" pad="2"/>
+<contactref element="U$3" pad="2"/>
+<wire x1="-85.09" y1="-24.825" x2="-93.13" y2="-33.02" width="0" layer="19" extent="1-1"/>
+<wire x1="-75.35" y1="-25.4" x2="-85.09" y2="-24.825" width="0" layer="19" extent="1-1"/>
+<wire x1="-75.35" y1="-29.21" x2="-75.35" y2="-25.4" width="0" layer="19" extent="1-1"/>
+<wire x1="-66.04" y1="-13.3225" x2="-75.35" y2="-25.4" width="0" layer="19" extent="1-1"/>
+<wire x1="-64.77" y1="-13.3225" x2="-66.04" y2="-13.3225" width="0" layer="19" extent="1-1"/>
+<wire x1="-62.23" y1="-13.3225" x2="-64.77" y2="-13.3225" width="0" layer="19" extent="1-1"/>
+<wire x1="-58.42" y1="-12.065" x2="-62.23" y2="-13.3225" width="0" layer="19" extent="1-1"/>
 <wire x1="-53.34" y1="-12.065" x2="-58.42" y2="-12.065" width="0" layer="19" extent="1-1"/>
-<wire x1="-58.42" y1="-18.415" x2="-58.42" y2="-12.065" width="0" layer="19" extent="1-1"/>
+<wire x1="-58.42" y1="-18.415" x2="-62.23" y2="-13.3225" width="0" layer="19" extent="1-1"/>
 <wire x1="-53.34" y1="-18.415" x2="-58.42" y2="-18.415" width="0" layer="19" extent="1-1"/>
 <wire x1="-46.14" y1="-2.54" x2="-53.34" y2="-12.065" width="0" layer="19" extent="1-1"/>
+<wire x1="-77.47" y1="-9.5375" x2="-66.04" y2="-13.3225" width="0" layer="19" extent="1-1"/>
 <wire x1="-29.21" y1="11.43" x2="-46.14" y2="-2.54" width="0" layer="19" extent="1-1"/>
 <wire x1="-38.52" y1="24.13" x2="-29.21" y2="11.43" width="0" layer="19" extent="1-1"/>
@@
 <contactref element="U$1" pad="24"/>
 <contactref element="R1" pad="2"/>
-<contactref element="JP1" pad="4"/>
-<wire x1="-41.06" y1="44.45" x2="-61.976" y2="-8.89" width="0" layer="19" extent="1-1"/>
-<wire x1="-21.93" y1="34.77" x2="-41.06" y2="44.45" width="0" layer="19" extent="1-1"/>
+<wire x1="-41.06" y1="44.45" x2="-21.93" y2="34.77" width="0" layer="19" extent="1-1"/>
 </signal>
 <signal name="LED1">
@@
 <signal name="AIN1">
 <contactref element="U$1" pad="46"/>
+<contactref element="JP2" pad="5"/>
+<wire x1="-25.53" y1="28.73" x2="-74.93" y2="-13.3225" width="0" layer="19" extent="1-1"/>
 </signal>
 <signal name="AIN0">
 <contactref element="U$1" pad="45"/>
+<contactref element="JP2" pad="3"/>
+<wire x1="-25.13" y1="28.73" x2="-76.2" y2="-13.3225" width="0" layer="19" extent="1-1"/>
 </signal>
 <signal name="AIN2">
 <contactref element="U$1" pad="5"/>
+<contactref element="JP2" pad="7"/>
+<wire x1="-27.15" y1="31.15" x2="-73.66" y2="-13.3225" width="0" layer="19" extent="1-1"/>
 </signal>
 <signal name="AIN3">
 <contactref element="U$1" pad="6"/>
+<contactref element="JP2" pad="9"/>
+<wire x1="-27.15" y1="31.55" x2="-72.39" y2="-13.3225" width="0" layer="19" extent="1-1"/>
 </signal>
 <signal name="AIN4">
 <contactref element="U$1" pad="7"/>
+<contactref element="JP2" pad="10"/>
+<wire x1="-27.15" y1="31.95" x2="-72.39" y2="-9.5375" width="0" layer="19" extent="1-1"/>
 </signal>
 <signal name="AIN5">
 <contactref element="U$1" pad="8"/>
+<contactref element="JP2" pad="8"/>
+<wire x1="-27.15" y1="32.35" x2="-73.66" y2="-9.5375" width="0" layer="19" extent="1-1"/>
 </signal>
 <signal name="AIN6">
 <contactref element="U$1" pad="9"/>
+<contactref element="JP2" pad="6"/>
+<wire x1="-27.15" y1="32.75" x2="-74.93" y2="-9.5375" width="0" layer="19" extent="1-1"/>
 </signal>
 <signal name="AIN7">
 <contactref element="U$1" pad="10"/>
+<contactref element="JP2" pad="4"/>
+<wire x1="-27.15" y1="33.15" x2="-76.2" y2="-9.5375" width="0" layer="19" extent="1-1"/>
 </signal>
 <signal name="N$27">
@@
 <contactref element="U$1" pad="23"/>
 <contactref element="JP1" pad="2"/>
-<wire x1="-22.33" y1="34.77" x2="-61.976" y2="-6.35" width="0" layer="19" extent="1-1"/>
+<wire x1="-22.33" y1="34.77" x2="-67.31" y2="-9.5375" width="0" layer="19" extent="1-1"/>
 </signal>
 <signal name="N$6">
@@
 <contactref element="U$1" pad="38"/>
 <contactref element="U$2" pad="X2"/>
-<wire x1="-33.02" y1="22.86" x2="-22.33" y2="28.73" width="0" layer="19" extent="1-1"/>
+<wire x1="-34.71" y1="24.78" x2="-22.33" y2="28.73" width="0" layer="19" extent="1-1"/>
 </signal>
 <signal name="N$5">
 <contactref element="U$1" pad="37"/>
 <contactref element="U$2" pad="X1"/>
-<wire x1="-36.83" y1="26.67" x2="-21.93" y2="28.73" width="0" layer="19" extent="1-1"/>
+<wire x1="-36.41" y1="23.48" x2="-21.93" y2="28.73" width="0" layer="19" extent="1-1"/>
 </signal>
 <signal name="N$7">
 <contactref element="U$2" pad="GND2"/>
 <contactref element="C8" pad="1"/>
-<wire x1="-31.33" y1="44.45" x2="-36.83" y2="22.86" width="0" layer="19" extent="1-1"/>
+<wire x1="-31.33" y1="44.45" x2="-36.41" y2="24.78" width="0" layer="19" extent="1-1"/>
 </signal>
 <signal name="N$9">
 <contactref element="U$2" pad="GND"/>
 <contactref element="C7" pad="1"/>
-<wire x1="-33.02" y1="26.67" x2="-27.52" y2="44.45" width="0" layer="19" extent="1-1"/>
+<wire x1="-34.71" y1="23.48" x2="-27.52" y2="44.45" width="0" layer="19" extent="1-1"/>
 </signal>
 <signal name="N$16">
@@
 <contactref element="LED2" pad="A"/>
 <contactref element="JP1" pad="1"/>
+<contactref element="C10" pad="1"/>
 <contactref element="JP2" pad="1"/>
-<wire x1="-67.564" y1="-6.35" x2="-77.724" y2="-6.35" width="0" layer="19" extent="1-1"/>
-<wire x1="-58.42" y1="-3.29" x2="-67.564" y2="-6.35" width="0" layer="19" extent="1-1"/>
+<contactref element="C11" pad="1"/>
+<wire x1="-77.05" y1="-25.4" x2="-77.05" y2="-29.21" width="0" layer="19" extent="1-1"/>
+<wire x1="-77.47" y1="-13.3225" x2="-77.05" y2="-25.4" width="0" layer="19" extent="1-1"/>
+<wire x1="-67.31" y1="-13.3225" x2="-77.47" y2="-13.3225" width="0" layer="19" extent="1-1"/>
+<wire x1="-58.42" y1="-3.29" x2="-67.31" y2="-13.3225" width="0" layer="19" extent="1-1"/>
 <wire x1="-54.61" y1="-3.29" x2="-58.42" y2="-3.29" width="0" layer="19" extent="1-1"/>
 </signal>
@@
 <wire x1="-54.61" y1="-1.79" x2="-58" y2="-6.35" width="0" layer="19" extent="1-1"/>
 </signal>
-<signal name="N$17">
-<contactref element="JP2" pad="4"/>
-</signal>
-<signal name="N$20">
-<contactref element="JP2" pad="3"/>
-</signal>
-<signal name="N$21">
-<contactref element="JP2" pad="5"/>
+<signal name="SDWCLK">
+<contactref element="JP1" pad="4"/>
+</signal>
+<signal name="ANT2">
+<contactref element="U$1" pad="32"/>
+<contactref element="U$3" pad="3"/>
+<wire x1="-21.11" y1="31.15" x2="-85.59" y2="-24.825" width="0" layer="19" extent="1-1"/>
+</signal>
+<signal name="ANT1">
+<contactref element="U$1" pad="31"/>
+<contactref element="U$3" pad="4"/>
+<wire x1="-21.11" y1="31.55" x2="-85.59" y2="-25.975" width="0" layer="19" extent="1-1"/>
+</signal>
+<signal name="VDD_PA">
+<contactref element="U$1" pad="30"/>
+<contactref element="U$3" pad="5"/>
+<contactref element="C12" pad="1"/>
+<wire x1="-85.09" y1="-25.975" x2="-94.83" y2="-33.02" width="0" layer="19" extent="1-1"/>
+<wire x1="-21.11" y1="31.95" x2="-85.09" y2="-25.975" width="0" layer="19" extent="1-1"/>
 </signal>
 <signal name="N$22">
-<contactref element="JP2" pad="7"/>
-</signal>
-<signal name="N$23">
-<contactref element="JP2" pad="9"/>
-</signal>
-<signal name="N$24">
-<contactref element="JP2" pad="6"/>
-</signal>
-<signal name="N$25">
-<contactref element="JP2" pad="8"/>
-</signal>
-<signal name="N$26">
-<contactref element="JP2" pad="10"/>
+<contactref element="U$3" pad="1"/>
+<contactref element="U$4" pad="FP"/>
+<wire x1="-84.59" y1="-24.825" x2="-94.41" y2="-25.4" width="0" layer="19" extent="1-1"/>
 </signal>
 </signals>

Commit message: Correccion Capacitores
Correccion de los capacitores C1 y C2 del Crystal
Connections:
- removed net N$7: C8.1, U$2.GND2
- removed net N$9: C7.1, U$2.GND
- net GND: now also C7.1, C8.1, U$2.GND, U$2.GND2; no longer C7.2, C8.2
- net N$4: now also C8.2
- net N$5: now also C7.2
Changed lines of the file:
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@@
 <contactref element="U$1" pad="34"/>
 <contactref element="C6" pad="2"/>
-<contactref element="C7" pad="2"/>
-<contactref element="C8" pad="2"/>
 <contactref element="BAT1" pad="2"/>
 <contactref element="C9" pad="2"/>
@@
 <contactref element="C12" pad="2"/>
 <contactref element="U$3" pad="2"/>
+<contactref element="U$2" pad="GND2"/>
+<contactref element="U$2" pad="GND"/>
+<contactref element="C8" pad="1"/>
+<contactref element="C7" pad="1"/>
 <wire x1="-85.09" y1="-24.825" x2="-93.13" y2="-33.02" width="0" layer="19" extent="1-1"/>
 <wire x1="-75.35" y1="-25.4" x2="-85.09" y2="-24.825" width="0" layer="19" extent="1-1"/>
@@
 <wire x1="-77.47" y1="-9.5375" x2="-66.04" y2="-13.3225" width="0" layer="19" extent="1-1"/>
 <wire x1="-29.21" y1="11.43" x2="-46.14" y2="-2.54" width="0" layer="19" extent="1-1"/>
-<wire x1="-38.52" y1="24.13" x2="-29.21" y2="11.43" width="0" layer="19" extent="1-1"/>
+<wire x1="-34.71" y1="23.48" x2="-29.21" y2="11.43" width="0" layer="19" extent="1-1"/>
+<wire x1="-36.41" y1="24.78" x2="-34.71" y2="23.48" width="0" layer="19" extent="1-1"/>
+<wire x1="-38.52" y1="24.13" x2="-36.41" y2="24.78" width="0" layer="19" extent="1-1"/>
 <wire x1="-42.33" y1="24.13" x2="-38.52" y2="24.13" width="0" layer="19" extent="1-1"/>
 <wire x1="-46.14" y1="24.13" x2="-42.33" y2="24.13" width="0" layer="19" extent="1-1"/>
-<wire x1="-27.15" y1="30.35" x2="-38.52" y2="24.13" width="0" layer="19" extent="1-1"/>
+<wire x1="-27.15" y1="30.35" x2="-34.71" y2="23.48" width="0" layer="19" extent="1-1"/>
 <wire x1="-27.15" y1="30.75" x2="-27.15" y2="30.35" width="0" layer="19" extent="1-1"/>
 <wire x1="-24.73" y1="28.73" x2="-27.15" y2="30.35" width="0" layer="19" extent="1-1"/>
@@
 <wire x1="-24.13" y1="31.75" x2="-24.33" y2="28.73" width="0" layer="19" extent="1-1"/>
 <wire x1="-26.33" y1="34.77" x2="-24.13" y2="31.75" width="0" layer="19" extent="1-1"/>
-<wire x1="-25.82" y1="44.45" x2="-26.33" y2="34.77" width="0" layer="19" extent="1-1"/>
-<wire x1="-22.01" y1="44.45" x2="-25.82" y2="44.45" width="0" layer="19" extent="1-1"/>
+<wire x1="-27.52" y1="44.45" x2="-26.33" y2="34.77" width="0" layer="19" extent="1-1"/>
+<wire x1="-31.33" y1="44.45" x2="-27.52" y2="44.45" width="0" layer="19" extent="1-1"/>
+<wire x1="-22.01" y1="44.45" x2="-27.52" y2="44.45" width="0" layer="19" extent="1-1"/>
 <wire x1="-18.2" y1="44.45" x2="-22.01" y2="44.45" width="0" layer="19" extent="1-1"/>
 <wire x1="-14.39" y1="44.45" x2="-18.2" y2="44.45" width="0" layer="19" extent="1-1"/>
-<wire x1="-29.63" y1="44.45" x2="-25.82" y2="44.45" width="0" layer="19" extent="1-1"/>
-<wire x1="-42.76" y1="44.45" x2="-29.63" y2="44.45" width="0" layer="19" extent="1-1"/>
+<wire x1="-42.76" y1="44.45" x2="-31.33" y2="44.45" width="0" layer="19" extent="1-1"/>
 </signal>
 <signal name="SWDCLK">
@@
 <contactref element="U$1" pad="38"/>
 <contactref element="U$2" pad="X2"/>
+<contactref element="C8" pad="2"/>
+<wire x1="-22.33" y1="28.73" x2="-29.63" y2="44.45" width="0" layer="19" extent="1-1"/>
 <wire x1="-34.71" y1="24.78" x2="-22.33" y2="28.73" width="0" layer="19" extent="1-1"/>
 </signal>
@@
 <contactref element="U$1" pad="37"/>
 <contactref element="U$2" pad="X1"/>
+<contactref element="C7" pad="2"/>
+<wire x1="-21.93" y1="28.73" x2="-25.82" y2="44.45" width="0" layer="19" extent="1-1"/>
 <wire x1="-36.41" y1="23.48" x2="-21.93" y2="28.73" width="0" layer="19" extent="1-1"/>
 </signal>
-<signal name="N$7">
-<contactref element="U$2" pad="GND2"/>
-<contactref element="C8" pad="1"/>
-<wire x1="-31.33" y1="44.45" x2="-36.41" y2="24.78" width="0" layer="19" extent="1-1"/>
-</signal>
-<signal name="N$9">
-<contactref element="U$2" pad="GND"/>
-<contactref element="C7" pad="1"/>
-<wire x1="-34.71" y1="23.48" x2="-27.52" y2="44.45" width="0" layer="19" extent="1-1"/>
-</signal>
 <signal name="N$16">

Commit message: Board 90%
Parts:
- removed BAT1: (no value), SparkFun-Electromechanical:BATTCON_20MM
- removed JP1: PROG-JLINK-SEAGGER, NordicSemi:M50-3600742
- removed JP2: PIN_HEADER_IO, NordicSemi:M50-3600742
- removed S1, S2: (no value), SparkFun-Electromechanical:TACTILE_SWITCH_SMD
- removed U$1: NRF51822, NordicSemi:QFN48
- removed U$2: CRYSTAL2.5X2, NordicSemi:2.5X2MM
- removed U$3: BALUN-2450BM, NordicSemi:2450BM14A0002
- removed U$4: ANTENA-2450AT, NordicSemi:2450AT18B100
- added ANT: ANTENA-2450AT, NordicSemi:2450AT18B100
- added BATT: 20mm coincell, SparkFun-Electromechanical:BATTCON_20MM_4LEGS_OVERPASTE
- added BLN: BALUN-2450BM, NordicSemi:2450BM14A0002
- added EXP: PIN_HEADER_IO, NordicSemi:M50-3600742
- added JP: JUMP_SMD, NordicSemi:JUMP-0.1-SMD
- added NRF51822: NRF51822, NordicSemi:QFN48
- added PROG: PROG-JLINK-SEAGGER, NordicSemi:M50-3600742
- added SW1: SWITCH_SMD_BB, NordicSemi:SWITCH3X2.5
- added SW2: SW1, NordicSemi:SWITCH3X2.5
- added XT: CRYSTAL2.5X2, NordicSemi:2.5X2MM
- moved C12 138.8 mm to (37.9, 10.5), turned to 270 degrees
- moved C11 110.2 mm to (27.8, 7.29), turned to 180 degrees
- moved C10 108.6 mm to (27.8, 5.77), turned to 180 degrees
- moved LED2 92.0 mm to (33.4, 3.30)
- moved R3 91.8 mm to (33.4, 6.55), turned to 90 degrees
- moved R2 89.9 mm to (31.9, 6.55), turned to 90 degrees
- moved LED1 86.7 mm to (31.9, 3.30)
- moved R1 85.6 mm to (34.9, 6.55), turned to 90 degrees
- moved C3 79.3 mm to (30.3, 6.55), turned to 270 degrees
- moved C1 77.4 mm to (37.6, 16.3)
- moved D1 76.5 mm to (22.0, 22.3)
- moved C2 70.0 mm to (26.5, 18.4)
- moved C9 69.9 mm to (18.5, 21.8), turned to 90 degrees
- moved L2 66.9 mm to (22.6, 16.2)
- moved C7 66.0 mm to (35.9, 23.7), turned to 315 degrees
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Connections:
- new net N$7: D1.2, JP.2
- net AIN0: now also EXP.3, NRF51822.45; no longer JP2.3, U$1.45
- net AIN1: now also EXP.5, NRF51822.46; no longer JP2.5, U$1.46
- net AIN2: now also EXP.7, NRF51822.5; no longer JP2.7, U$1.5
- net AIN3: now also EXP.9, NRF51822.6; no longer JP2.9, U$1.6
- net AIN4: now also EXP.10, NRF51822.7; no longer JP2.10, U$1.7
- net AIN5: now also EXP.8, NRF51822.8; no longer JP2.8, U$1.8
- net AIN6: now also EXP.6, NRF51822.9; no longer JP2.6, U$1.9
- net AIN7: now also EXP.4, NRF51822.10; no longer JP2.4, U$1.10
- net ANT1: now also BLN.4, NRF51822.31; no longer U$1.31, U$3.4
- net ANT2: now also BLN.3, NRF51822.32; no longer U$1.32, U$3.3
- net AVDD: now also NRF51822.35, NRF51822.36; no longer U$1.35, U$1.36
- net GND: now also BATT.2, BLN.2, EXP.2, NRF51822.13, NRF51822.3, NRF51822.33, NRF51822.34, NRF51822.4, NRF51822.GND, PROG.3, PROG.5, PROG.9, SW1.1, SW2.1, XT.GND, XT.GND2; no longer BAT1.2, JP1.3, JP1.5, JP1.9, JP2.2, S1.1, S1.2, S2.1, S2.2, U$1.13, U$1.3, U$1.33, U$1.34, U$1.4, U$1.40, U$1.41, U$1.42, U$1.43, U$1.44, U$1.GND, U$2.GND, U$2.GND2, U$3.2
- net LED1: now also NRF51822.14; no longer U$1.14
- net LED2: now also NRF51822.15; no longer U$1.15
- net N$1: now also NRF51822.39; no longer U$1.39
- net N$10: now also NRF51822.16; no longer U$1.16
- net N$11: now also NRF51822.17; no longer U$1.17
- net N$12: now also NRF51822.18; no longer U$1.18
- net N$13: now also NRF51822.19; no longer U$1.19
- net N$14: now also NRF51822.20; no longer U$1.20
- net N$15: now also NRF51822.21; no longer U$1.21
- net N$16: now also BATT.1, JP.1; no longer BAT1.1, D1.2
- net N$22: now also ANT.FP, BLN.1; no longer U$3.1, U$4.FP
- net N$27: now also NRF51822.11; no longer U$1.11
- net N$28: now also NRF51822.25; no longer U$1.25
- net N$29: now also NRF51822.26; no longer U$1.26
- net N$3: now also NRF51822.2; no longer U$1.2
- net N$30: now also NRF51822.27; no longer U$1.27
- net N$31: now also NRF51822.28; no longer U$1.28
- net N$4: now also NRF51822.38, XT.X2; no longer U$1.38, U$2.X2
- net N$5: now also NRF51822.37, XT.X1; no longer U$1.37, U$2.X1
- net N$6: now also NRF51822.29; no longer U$1.29
- net N$8: now also NRF51822.22; no longer U$1.22
- net SDWCLK: now also PROG.4; no longer JP1.4
- net SW1: now also NRF51822.48, SW1.2; no longer S1.3, S1.4, U$1.48
- net SW2: now also NRF51822.47, SW2.2; no longer S2.3, S2.4, U$1.47
- net SWDCLK: now also NRF51822.24; no longer U$1.24
- net SWDIO: now also NRF51822.23, PROG.2; no longer JP1.2, U$1.23
- net VCC: now also EXP.1, PROG.1; no longer JP1.1, JP2.1
- net VCC_NRF: now also NRF51822.1, NRF51822.12; no longer U$1.1, U$1.12
- net VDD_PA: now also BLN.5, NRF51822.30; no longer U$1.30, U$3.5
Routing:
- net VCC_NRF: track 0.00 -> 33.0 mm, vias 0 -> 3
- net AIN0: track 0.00 -> 31.4 mm
- net AVDD: track 0.00 -> 29.1 mm, vias 0 -> 2
- net AIN1: track 0.00 -> 28.8 mm
- net N$20: track 0.00 -> 20.7 mm
- net AIN2: track 0.00 -> 18.3 mm
- net AIN3: track 0.00 -> 16.4 mm
- net N$9: track 0.00 -> 15.9 mm
- net VCC: track 0.00 -> 15.5 mm
- net SWDIO: track 0.00 -> 12.8 mm, vias 0 -> 2
- net SW2: track 0.00 -> 11.8 mm, vias 0 -> 2
- net SW1: track 0.00 -> 9.47 mm, vias 0 -> 2
- net AIN4: track 0.00 -> 8.41 mm
- net AIN7: track 0.00 -> 8.29 mm
- net N$4: track 0.00 -> 8.16 mm
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- added copper zone on layer 1, net GND
- added copper zone on layer 16, net GND
Other:
- board size 160 x 100 mm -> 47 x 27.9 mm
- board text added: "Bluetooth 4.0 Low Energy"

Commit message: BLE NRF51822v1
Board 100%, Lbr update Top places
Parts:
- moved ANT 0.34 mm to (43.3, 14.3)
- moved C5 0.05 mm to (37.6, 17.8)
- moved C1 0.05 mm to (37.6, 16.3)
Connections:
- new net N$17: NRF51822.3
- new net N$21: NRF51822.4
- new net N$24: NRF51822.44
- new net N$25: NRF51822.43
- new net N$26: NRF51822.42
- new net N$32: NRF51822.41
- new net N$33: NRF51822.40
- net GND: no longer NRF51822.3, NRF51822.4
Routing:
- net N$23: track 0.00 -> 9.93 mm
- net N$20: track 20.7 -> 11.1 mm
- net VDD_PA: track 5.33 -> 4.76 mm
Other:
- board text added: "BLE NRF51822v1"
- board text added: "Bluetooth"
- board text added: "SMART"
- board text added: "Stratia"
- board text removed: "Bluetooth 4.0 Low Energy"
