File: nRF51822.brd (EAGLE design)
At the start: 47 x 27.9 mm, 30 parts, among them SW1 SWITCH_SMD_BB, SW2 SW1

Commit message: Esquemático Rev 2
Parts:
- removed D1: BAT165, SparkFun-DiscreteSemi:SOD-323
- removed EXP: PIN_HEADER_IO, NordicSemi:M50-3600742
- removed JP: JUMP_SMD, NordicSemi:JUMP-0.1-SMD
- added C13, C14: 12pF, SparkFun-Capacitors:0603-CAP
- added JP1: CM, NordicSemi:JUMP-0.05-SMD
- added JP2: VCC_PROG, NordicSemi:JUMP-0.05-SMD
- added P0, P1, P2, P3, P4, P5, P6, P7: TPB1,27, testpad:B1,27
- added R4, R5: 4.7K, SparkFun-Resistors:0603-RES
- added R6, R8: 150, SparkFun-Resistors:0603-RES
- added R7, R9: 10K, SparkFun-Resistors:0603-RES
- added T1, T2: BC847, transistor:SOT23
- added Y1: CRYSTAL.ABS07, abracon:ABS07
- R2, R3: value 100 -> 150
- SW2: value SW1 -> SWITCH_SMD_BB
Connections:
- removed net AIN0: EXP.3, NRF51822.45
- removed net AIN1: EXP.5, NRF51822.46
- removed net AIN2: EXP.7, NRF51822.5
- removed net AIN3: EXP.9, NRF51822.6
- removed net AIN4: EXP.10, NRF51822.7
- removed net AIN5: EXP.8, NRF51822.8
- removed net AIN6: EXP.6, NRF51822.9
- removed net AIN7: EXP.4, NRF51822.10
- removed net N$27 (its old number): NRF51822.11
- removed net SDWCLK: PROG.4
- removed net VCC_NRF: C2.1, C3.1, C9.1, D1.1, NRF51822.1, NRF51822.12
- new net N$17: R3.2, T2.3
- new net N$19: R8.2, R9.2, SW2.2
- new net N$34: R4.2, T1.1
- new net N$35: R6.2, R7.2, SW1.2
- new net P00: NRF51822.4, P0.TP
- new net P01: NRF51822.5, P1.TP
- new net P02: NRF51822.6, P2.TP
- new net P03: NRF51822.7, P3.TP
- new net P04: NRF51822.8, P4.TP
- new net P05: NRF51822.9, P5.TP
- new net P06: NRF51822.10, P6.TP
- new net P07: NRF51822.11, P7.TP
- new net XL1: C13.1, NRF51822.45, Y1.2
- new net XL2: C14.1, NRF51822.46, Y1.1
- net GND: now also C13.2, C14.2, JP2.P$2, T1.2, T2.2; no longer EXP.2
- net LED1: now also R4.1; no longer R2.2
- net LED2: now also R5.1; no longer R3.2
- net N$16: now also JP1.P$1; no longer JP.1
- net N$21: now also R2.2, T1.3; no longer NRF51822.4
- net N$7: now also R5.2, T2.1; no longer D1.2, JP.2
- net SW1: now also R6.1; no longer SW1.2
- net SW2: now also R8.1; no longer SW2.2
- net SWDCLK: now also PROG.4
- net VCC: now also C2.1, C3.1, C9.1, JP1.P$2, JP2.P$1, NRF51822.1, NRF51822.12, R7.1, R9.1; no longer EXP.1
Routing:
- net VCC_NRF: track 33.0 -> 0.00 mm, vias 3 -> 0
- net AIN0: track 31.2 -> 0.00 mm
- net AIN1: track 29.0 -> 0.00 mm
- net AIN2: track 18.4 -> 0.00 mm
- net AIN3: track 16.5 -> 0.00 mm
- net AIN4: track 8.76 -> 0.00 mm
- net AIN7: track 8.14 -> 0.00 mm
- net AIN5: track 7.92 -> 0.00 mm
- net AIN6: track 7.78 -> 0.00 mm
- net VCC: track 15.5 -> 9.83 mm
- net N$7: track 4.49 -> 0.00 mm
- net N$27: track 1.65 -> 0.00 mm
- net N$18: track 1.65 -> 0.00 mm
- net SW2: track 11.7 -> 10.5 mm
- net SW1: track 9.32 -> 8.18 mm
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
Commit message: Board V2 - 85%
Parts:
- moved JP2 90.0 mm to (18.7, 10.5), turned to 270 degrees
- moved P7 85.4 mm to (23.9, 8.33)
- moved P6 81.8 mm to (21.8, 9.19)
- moved P5 79.4 mm to (23.9, 10.1)
- moved P4 75.8 mm to (21.8, 10.9)
- moved P3 73.4 mm to (23.9, 11.8)
- moved R9 70.3 mm to (23.6, 25.0), turned to 90 degrees
- moved P2 69.8 mm to (21.8, 12.6)
- moved P1 67.5 mm to (23.9, 13.5)
- moved R8 66.1 mm to (19.2, 25.0), turned to 270 degrees
- moved R7 65.2 mm to (25.3, 25.0), turned to 90 degrees
- moved R6 64.4 mm to (29.7, 25.0), turned to 270 degrees
- moved P0 64.0 mm to (21.8, 14.4)
- moved R5 48.5 mm to (33.4, 6.55), turned to 270 degrees
- moved R4 45.2 mm to (31.9, 6.55), turned to 270 degrees
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Routing:
- net VCC: track 9.83 -> 30.8 mm
- net XL1: track 0.00 -> 9.13 mm
- net P06: track 0.00 -> 8.46 mm
- net XL2: track 0.00 -> 8.19 mm
- net P04: track 0.00 -> 8.07 mm
- net P02: track 0.00 -> 7.69 mm
- net SW2: track 10.5 -> 17.9 mm
- net P00: track 0.00 -> 7.38 mm
- net N$35: track 0.00 -> 6.74 mm
- net N$19: track 0.00 -> 6.72 mm
- net P07: track 0.00 -> 6.62 mm
- net AVDD: track 28.9 -> 35.5 mm
- net P05: track 0.00 -> 6.24 mm
- net P03: track 0.00 -> 5.85 mm
- net P01: track 0.00 -> 5.47 mm
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